Commit message: add fixed google robot urdf to avoid mesh penetration between shoulder and base

File: mani_skill2/assets/descriptions/googlerobot_description/meta_sim_fix_wheel.urdf (robot description, URDF)
Before this commit: robot meta, 34 links, 33 joints
Links:
- added link link_rear_wheel_left; collision mesh filename=coarse_meshes/link_rear_wheel.glb; visual mesh filename=coarse_meshes/link_rear_wheel.glb
- added link link_rear_wheel_right; collision mesh filename=coarse_meshes/link_rear_wheel.glb; visual mesh filename=coarse_meshes/link_rear_wheel.glb
- link link_base: geometry collision mesh filename=coarse_meshes/link_base_0.glb; collision mesh filename=coarse_meshes/link_base_1.glb
Joints:
- added joint joint_rear_wheel_left: type fixed, parent link_base, child link_rear_wheel_left, origin xyz=-0.338371 0.094989 -0.029296 rpy=0 0 0, axis 0 1 0, limit lower=-inf upper=inf effort=10.0 velocity=12.9
- added joint joint_rear_wheel_right: type fixed, parent link_base, child link_rear_wheel_right, origin xyz=-0.338371 -0.094989 -0.029296 rpy=0 0 0, axis 0 1 0, limit lower=-inf upper=inf effort=10.0 velocity=12.9
- joint joint_wheel_left: limit (none) -> lower=-inf upper=inf effort=10.0 velocity=12.9
- joint joint_wheel_right: limit (none) -> lower=-inf upper=inf effort=10.0 velocity=12.9

File: mani_skill2/assets/descriptions/googlerobot_description_old/meta_sim.urdf (robot description, URDF)
Before this commit: robot meta, 36 links, 35 joints
Links:
- removed link link_rear_wheel_left
- removed link link_rear_wheel_right
- link link_base: geometry collision mesh filename=coarse_meshes/link_base_part_0_vhacd.obj; collision mesh filename=coarse_meshes/link_base_part_1_vhacd.obj
Joints:
- removed joint joint_rear_wheel_left
- removed joint joint_rear_wheel_right

File: mani_skill2/assets/descriptions/googlerobot_description_old/meta_sim_fix_wheel.urdf (robot description, URDF)
Before this commit: robot meta, 36 links, 35 joints
Links:
- removed link link_rear_wheel_left
- removed link link_rear_wheel_right
- link link_base: geometry collision mesh filename=coarse_meshes/link_base_part_0_vhacd.obj; collision mesh filename=coarse_meshes/link_base_part_1_vhacd.obj
Joints:
- removed joint joint_rear_wheel_left
- removed joint joint_rear_wheel_right
- joint joint_wheel_left: limit lower=-inf upper=inf effort=10.0 velocity=12.9 -> (none); type continuous -> fixed
- joint joint_wheel_right: limit lower=-inf upper=inf effort=10.0 velocity=12.9 -> (none); type continuous -> fixed
