Commit message: (1) Env enable_tgs=True to prevent mesh penetration; (2) remove finger tip joint; modify urdf such that finger tip joint is always at an angle wrt finger link to simulate real grasping

File: mani_skill2/assets/descriptions/googlerobot_description/google_robot_meta_sim_fix_fingertip.urdf (robot description, URDF)
Before this commit: robot meta, 36 links, 35 joints
Joints:
- joint joint_finger_tip_left: axis 1 0 0 -> (none); limit lower=0.0 upper=1.2 -> (none); origin xyz=8.68878191722553E-19 -1.03567252152576E-02 6.41556076619853E-02 rpy=0 0 0 -> xyz=8.68878191722553E-19 -1.03567252152576E-02 6.41556076619853E-02 rpy=0.6 0 0; type revolute -> fixed
- joint joint_finger_tip_right: axis 1 0 0 -> (none); limit lower=0.0 upper=1.2 -> (none); origin xyz=8.68878191722553E-19 -1.03567252152576E-02 6.41556076619853E-02 rpy=0 0 0 -> xyz=8.68878191722553E-19 -1.03567252152576E-02 6.41556076619853E-02 rpy=0.6 0 0; type revolute -> fixed
- joint joint_rear_wheel_left: type fixed -> continuous
- joint joint_rear_wheel_right: type fixed -> continuous
- joint joint_wheel_left: type fixed -> continuous
- joint joint_wheel_right: type fixed -> continuous

File: mani_skill2/assets/descriptions/googlerobot_description/google_robot_meta_sim_fix_wheel_fix_fingertip.urdf (robot description, URDF)
Before this commit: robot meta, 36 links, 35 joints
Joints:
- joint joint_finger_tip_left: axis 1 0 0 -> (none); limit lower=0.0 upper=1.2 -> (none); origin xyz=8.68878191722553E-19 -1.03567252152576E-02 6.41556076619853E-02 rpy=0 0 0 -> xyz=8.68878191722553E-19 -1.03567252152576E-02 6.41556076619853E-02 rpy=0.6 0 0; type revolute -> fixed
- joint joint_finger_tip_right: axis 1 0 0 -> (none); limit lower=0.0 upper=1.2 -> (none); origin xyz=8.68878191722553E-19 -1.03567252152576E-02 6.41556076619853E-02 rpy=0 0 0 -> xyz=8.68878191722553E-19 -1.03567252152576E-02 6.41556076619853E-02 rpy=0.6 0 0; type revolute -> fixed
- joint joint_rear_wheel_left: type continuous -> fixed
- joint joint_rear_wheel_right: type continuous -> fixed
- joint joint_wheel_left: type continuous -> fixed
- joint joint_wheel_right: type continuous -> fixed

Commit message: (1) modify urdf tcp pose; (2) adjust pd based on mujoco xml; (3) fix gripper controller; (4) add more envs

File: mani_skill2/assets/descriptions/googlerobot_description/google_robot_meta_sim_fix_fingertip.urdf (robot description, URDF)
Before this commit: robot meta, 36 links, 35 joints
Links:
- added link link_base_inertial
Joints:
- added joint link_base_inertial_joint: type fixed, parent link_base, child link_base_inertial, origin xyz=-0.142542994624505 2.33339305547787E-03 0.130110970092973 rpy=0 0 0
- joint gripper_tcp_joint: origin xyz=0 0 0.15 rpy=0 0 0 -> xyz=4.3374896E-03 1.8852949E-03 1.6353297E-01 rpy=-0.001328879239766479 -0.00443973089771006 -0.0008686511567993004
- joint joint_finger_tip_left: origin xyz=8.68878191722553E-19 -1.03567252152576E-02 6.41556076619853E-02 rpy=0.6 0 0 -> xyz=8.68878191722553E-19 -1.03567252152576E-02 6.41556076619853E-02 rpy=0.45 0 0
- joint joint_finger_tip_right: origin xyz=8.68878191722553E-19 -1.03567252152576E-02 6.41556076619853E-02 rpy=0.6 0 0 -> xyz=8.68878191722553E-19 -1.03567252152576E-02 6.41556076619853E-02 rpy=0.45 0 0

File: mani_skill2/assets/descriptions/googlerobot_description/google_robot_meta_sim_fix_wheel_fix_fingertip.urdf (robot description, URDF)
Before this commit: robot meta, 36 links, 35 joints
Links:
- added link link_base_inertial
Joints:
- added joint link_base_inertial_joint: type fixed, parent link_base, child link_base_inertial, origin xyz=-0.142542994624505 2.33339305547787E-03 0.130110970092973 rpy=0 0 0
- joint gripper_tcp_joint: origin xyz=0 0 0.15 rpy=0 0 0 -> xyz=4.3374896E-03 1.8852949E-03 1.6353297E-01 rpy=-0.001328879239766479 -0.00443973089771006 -0.0008686511567993004
- joint joint_finger_tip_left: origin xyz=8.68878191722553E-19 -1.03567252152576E-02 6.41556076619853E-02 rpy=0.6 0 0 -> xyz=8.68878191722553E-19 -1.03567252152576E-02 6.41556076619853E-02 rpy=0.45 0 0
- joint joint_finger_tip_right: origin xyz=8.68878191722553E-19 -1.03567252152576E-02 6.41556076619853E-02 rpy=0.6 0 0 -> xyz=8.68878191722553E-19 -1.03567252152576E-02 6.41556076619853E-02 rpy=0.45 0 0
