Commit message: add and refactor visual matching google robot urdfs

File: mani_skill2/assets/descriptions/googlerobot_description/google_robot_meta_sim_fix_wheel_fix_fingertip_recolor_cabinet_visual_matching_1.urdf (robot description, URDF)
Before this commit: robot meta, 37 links, 36 joints
Links:
- link link_base: geometry collision mesh filename=coarse_meshes/link_base_0.glb; collision mesh filename=coarse_meshes/link_base_1.glb
- link link_bicep: geometry collision mesh filename=coarse_meshes/link_bicep_vhacd.obj; visual mesh filename=3obj_recolor_cabinet_visual_matching_1/link_bicep.3obj.obj
- link link_elbow: geometry collision mesh filename=coarse_meshes/link_elbow_vhacd.obj; visual mesh filename=3obj_recolor_cabinet_visual_matching_1/link_elbow.3obj.obj
- link link_finger_left: geometry collision mesh filename=coarse_meshes/link_finger_base_boxified.obj; visual mesh filename=3obj_recolor_cabinet_visual_matching_1/link_finger_base_sim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
- link link_finger_right: geometry collision mesh filename=coarse_meshes/link_finger_base_boxified.obj; visual mesh filename=3obj_recolor_cabinet_visual_matching_1/link_finger_base_sim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
- link link_finger_tip_left: geometry collision mesh filename=coarse_meshes/link_finger_tip_boxified.obj; visual mesh filename=3obj_recolor_cabinet_visual_matching_1/link_finger_tip_simp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
- link link_finger_tip_right: geometry collision mesh filename=coarse_meshes/link_finger_tip_boxified.obj; visual mesh filename=3obj_recolor_cabinet_visual_matching_1/link_finger_tip_simp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
- link link_forearm: geometry collision mesh filename=coarse_meshes/link_forearm_vhacd.obj; visual mesh filename=3obj_recolor_cabinet_visual_matching_1/link_forearm.3obj.obj
- link link_gripper: geometry collision mesh filename=coarse_meshes/link_gripper_vhacd.obj; visual mesh filename=3obj_recolor_cabinet_visual_matching_1/link_gripper.3obj.obj
- link link_shoulder: geometry collision mesh filename=coarse_meshes/link_shoulder_vhacd.obj; visual mesh filename=3obj_recolor_cabinet_visual_matching_1/link_shoulder.3obj.o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
- link link_wrist: geometry collision mesh filename=coarse_meshes/link_wrist_vhacd.obj; visual mesh filename=3obj_recolor_cabinet_visual_matching_1/link_wrist.3obj.obj

File: mani_skill2/assets/descriptions/googlerobot_description/google_robot_meta_sim_fix_wheel_fix_fingertip_recolor_cabinet_visual_matching_gripper_only.urdf (robot description, URDF)
Before this commit: robot meta, 37 links, 36 joints
Links:
- link link_base: geometry collision mesh filename=coarse_meshes/link_base_0.glb; collision mesh filename=coarse_meshes/link_base_1.glb
- link link_finger_left: geometry collision mesh filename=coarse_meshes/link_finger_base_boxified.obj; visual mesh filename=3obj_recolor_cabinet_visual_matching_gripper_only/link_fing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
- link link_finger_right: geometry collision mesh filename=coarse_meshes/link_finger_base_boxified.obj; visual mesh filename=3obj_recolor_cabinet_visual_matching_gripper_only/link_fing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
- link link_finger_tip_left: geometry collision mesh filename=coarse_meshes/link_finger_tip_boxified.obj; visual mesh filename=3obj_recolor_cabinet_visual_matching_gripper_only/link_fing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
- link link_finger_tip_right: geometry collision mesh filename=coarse_meshes/link_finger_tip_boxified.obj; visual mesh filename=3obj_recolor_cabinet_visual_matching_gripper_only/link_fing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
