Commit message: Update drawer tasks
* use white interior, add handles, adjust intervals for mk_station.urdf
* replace a1 with a2
* change lighting

File: data/custom/mk_station.urdf (robot description, URDF)
Before this commit: robot mk_station, 4 links, 3 joints
Links:
- link bottom_drawer: geometry collision box size=0.015000 0.61500 0.14000; collision box size=0.02000 0.51500 0.10000
- link middle_drawer: geometry collision box size=0.015000 0.61500 0.14000; collision box size=0.02000 0.51500 0.10000
- link top_drawer: geometry collision box size=0.015000 0.61500 0.14000; collision box size=0.02000 0.51500 0.10000
Joints:
- joint bottom_drawer_joint: origin xyz=0.00000 0.00000 0.16500 rpy=0.00000 0.00000 0.00000 -> xyz=0.00000 0.00000 0.17800 rpy=0.00000 0.00000 0.00000
- joint middle_drawer_joint: origin xyz=0.00000 0.00000 0.41000 rpy=0.00000 0.00000 0.00000 -> xyz=0.00000 0.00000 0.42300 rpy=0.00000 0.00000 0.00000
- joint top_drawer_joint: origin xyz=0.00000 0.00000 0.65500 rpy=0.00000 0.00000 0.00000 -> xyz=0.00000 0.00000 0.66800 rpy=0.00000 0.00000 0.00000
