Commit message: update widowx descriptions and missing files

File: mani_skill2/assets/descriptions/widowx_description/wx250s.urdf (robot description, URDF)
Before this commit: robot wx250s, 14 links, 13 joints
Joints:
- joint elbow: limit lower=-3.21 upper=4.29 effort=100 velocity=3.141592653589793 -> lower=-2.1467549799530254 upper=1.6057029118347832 effort=15 velocity=3.141592653589793; origin xyz=0.04975 0 0.25 rpy=3.141592653589793 0 0 -> xyz=0.04975 0 0.25 rpy=0 0 0
- joint forearm_roll: limit lower=-6.28318530718 upper=6.28318530718 effort=100 velocity=3.141592653589793 -> lower=-3.141582653589793 upper=3.141582653589793 effort=2 velocity=3.141592653589793
- joint left_finger: limit lower=0.015 upper=0.037 effort=10 velocity=1 -> lower=0.015 upper=0.037 effort=5 velocity=1
- joint right_finger: limit lower=0.015 upper=0.037 effort=10 velocity=1 -> lower=0.015 upper=0.037 effort=5 velocity=1
- joint shoulder: limit lower=-3.77 upper=3.98 effort=100 velocity=3.141592653589793 -> lower=-1.8849555921538759 upper=1.9896753472735358 effort=20 velocity=3.141592653589793
- joint waist: limit lower=-6.28318530718 upper=6.28318530718 effort=100 velocity=3.141592653589793 -> lower=-3.141592653589793 upper=3.141592653589793 effort=10 velocity=3.141592653589793; origin xyz=0 0 0.0716 rpy=0 0 0 -> xyz=0 0 0.072 rpy=0 0 0
- joint wrist_angle: limit lower=-4.30 upper=3.49 effort=100 velocity=3.141592653589793 -> lower=-1.7453292519943295 upper=2.1467549799530254 effort=5 velocity=3.141592653589793
- joint wrist_rotate: limit lower=-6.28318530718 upper=6.28318530718 effort=100 velocity=3.141592653589793 -> lower=-3.141582653589793 upper=3.141582653589793 effort=1 velocity=3.141592653589793; origin xyz=0.065 0 0 rpy=-3.141592653589793 0 0 -> xyz=0.065 0 0 rpy=0 0 0

Commit message: update bridge widowx urdf to use gripper bar collision mesh but ignore its collision w/ finger links; refine sink mesh in bridge eggplant env

File: mani_skill2/assets/descriptions/widowx_description/wx250s.urdf (robot description, URDF)
Before this commit: robot wx250s, 14 links, 13 joints
Links:
- link gripper_bar_link: geometry collision mesh filename=meshes_wx250s/WXSA-250-M-9-Gripper-Bar.stl scale=0.001 0.001 0.001; visual mesh filename=meshes_wx250s/WXSA-250-M-9-Gripper-Bar.obj scale=0.001 0.001 0.001
